Commit message: moveit cyton alpha

File: cyton_alpha_description/urdf/cyton_alpha.structure.xacro (robot description, xacro)
@@ -10,5 +10,6 @@
 				<mass
 					value="0.40583" />
-				<inertia
+				<inertia ixx="1.0" ixy="0.0" ixz="0.0" iyy="1.0" iyz="0.0" izz="1.0" />
+				<!-- <inertia
 					ixx="0.00082976"
 					ixy="8.1234E-05"
@@ -17,4 +18,5 @@
 					iyz="2.8245E-06"
 					izz="0.00086815" />
+				-->
 			</inertial>
 			<visual>

Commit message: Update to run on Indigo

File: cyton_alpha_description/urdf/cyton_alpha.structure.xacro (robot description, xacro)
@@ -567,7 +567,8 @@
 		<transmission name="shoulder_base_trans">
 			<type>transmission_interface/SimpleTransmission</type>
-			<joint name="shoulder_base"/>
+			<joint name="shoulder_base">
+				<hardwareInterface>EffortJointInterface</hardwareInterface>
+			</joint>
 			<actuator name="shoulder_base_motor">
-				<hardwareInterface>EffortJointInterface</hardwareInterface>
 				<mechanicalReduction>1</mechanicalReduction>
 			</actuator>
@@ -575,7 +576,8 @@
 		<transmission name="shoulder_pitch_trans">
 			<type>transmission_interface/SimpleTransmission</type>
-			<joint name="shoulder_pitch"/>
+			<joint name="shoulder_pitch">
+				<hardwareInterface>EffortJointInterface</hardwareInterface>
+			</joint>
 			<actuator name="shoulder_pitch_motor">
-				<hardwareInterface>EffortJointInterface</hardwareInterface>
 				<mechanicalReduction>1</mechanicalReduction>
 			</actuator>
@@ -583,7 +585,8 @@
 		<transmission name="shoulder_yaw_trans">
 			<type>transmission_interface/SimpleTransmission</type>
-			<joint name="shoulder_yaw"/>
+			<joint name="shoulder_yaw">
+				<hardwareInterface>EffortJointInterface</hardwareInterface>
+			</joint>
 			<actuator name="shoulder_yaw_motor">
-				<hardwareInterface>EffortJointInterface</hardwareInterface>
 				<mechanicalReduction>1</mechanicalReduction>
 			</actuator>
@@ -591,7 +594,8 @@
 		<transmission name="elbow_pitch_trans">
 			<type>transmission_interface/SimpleTransmission</type>
-			<joint name="elbow_pitch"/>
+			<joint name="elbow_pitch">
+				<hardwareInterface>EffortJointInterface</hardwareInterface>
+			</joint>
 			<actuator name="elbow_pitch_motor">
-				<hardwareInterface>EffortJointInterface</hardwareInterface>
 				<mechanicalReduction>1</mechanicalReduction>
 			</actuator>
@@ -599,7 +603,8 @@
 		<transmission name="wrist_roll_trans">
 			<type>transmission_interface/SimpleTransmission</type>
-			<joint name="wrist_roll"/>
+			<joint name="wrist_roll">
+				<hardwareInterface>EffortJointInterface</hardwareInterface>
+			</joint>
 			<actuator name="wrist_roll_motor">
-				<hardwareInterface>EffortJointInterface</hardwareInterface>
 				<mechanicalReduction>1</mechanicalReduction>
 			</actuator>
@@ -607,7 +612,8 @@
 		<transmission name="wrist_yaw_trans">
 			<type>transmission_interface/SimpleTransmission</type>
-			<joint name="wrist_yaw"/>
+			<joint name="wrist_yaw">
+				<hardwareInterface>EffortJointInterface</hardwareInterface>
+			</joint>
 			<actuator name="wrist_yaw_motor">
-				<hardwareInterface>EffortJointInterface</hardwareInterface>
 				<mechanicalReduction>1</mechanicalReduction>
 			</actuator>
@@ -615,7 +621,8 @@
 		<transmission name="wrist_pitch_trans">
 			<type>transmission_interface/SimpleTransmission</type>
-			<joint name="wrist_pitch"/>
+			<joint name="wrist_pitch">
+				<hardwareInterface>EffortJointInterface</hardwareInterface>
+			</joint>
 			<actuator name="wrist_pitch_motor">
-				<hardwareInterface>EffortJointInterface</hardwareInterface>
 				<mechanicalReduction>1</mechanicalReduction>
 			</actuator>
@@ -623,7 +630,8 @@
 		<transmission name="claw_left_trans">
 			<type>transmission_interface/SimpleTransmission</type>
-			<joint name="claw_left"/>
+			<joint name="claw_left">
+				<hardwareInterface>EffortJointInterface</hardwareInterface>
+			</joint>
 			<actuator name="claw_left_motor">
-				<hardwareInterface>EffortJointInterface</hardwareInterface>
 				<mechanicalReduction>1</mechanicalReduction>
 			</actuator>
@@ -631,7 +639,8 @@
 		<transmission name="claw_right_trans">
 			<type>transmission_interface/SimpleTransmission</type>
-			<joint name="claw_right"/>
+			<joint name="claw_right">
+				<hardwareInterface>EffortJointInterface</hardwareInterface>
+			</joint>
 			<actuator name="claw_right_motor">
-				<hardwareInterface>EffortJointInterface</hardwareInterface>
 				<mechanicalReduction>1</mechanicalReduction>
 			</actuator>

Commit message: Funcionando sem a junta do gripper

File: cyton_alpha_description/urdf/cyton_alpha.structure.xacro (robot description, xacro)
@@ -78,5 +78,5 @@
 					rpy="0 0 0" />
 				<geometry>
-					<box size="0.136 0.051 0.160"/>
+					<box size="0.136 0.051 0.10"/> <!--0.160-->
 				</geometry>
 			</collision>

Commit message: Adicionado joint virtual para grasp

File: cyton_alpha_description/urdf/cyton_alpha.structure.xacro (robot description, xacro)
@@ -1,4 +1,6 @@
 <?xml version="1.0"?>
 <robot xmlns:xacro="http://ros.org/wiki/xacro">
+	<!-- the grasp _frame need of this macro -  -->
+  <xacro:include filename="$(find cyton_alpha_description)/urdf/inertia_gripper.xacro" />
 	<xacro:macro name="cyton_alpha" params="name">
 		<link
@@ -394,4 +396,29 @@
 			</collision>
 		</link>
+		<!-- Grasping frame (to correct position of grasp) virtual -->
+	    <link
+	    	name="grasping_frame">
+	      	<inertial>
+	       		<origin
+	       			xyz="0 0 0"
+	       			rpy="0 0 0" />
+	        	<mass
+	        		value="0.0001" />
+	        	<cuboid_inertia
+	        	 	mass="0.0001"
+	        	 	x="0.001"
+	        	 	y="0.001"
+	        	 	z="0.001"/>
+	      </inertial>
+	    </link>
+	    <!--joint grasp frame - this joint stay on top of link7-->
+	    <joint
+	    	name="grasping_frame_joint"
+	    	type="fixed">
+	      <parent
+	      	link="link7"/>
+	      <child link="grasping_frame"/>
+	      <origin xyz="-0.02 0.05 0" rpy="-1.57 0 0"/>
+	    </joint>
 		<joint
 			name="shoulder_base"
